Commit message: Updated final codes

File: Task_1/volta_description/urdf/accessories/lidar_volta.urdf.xacro (robot description, xacro)
@@ -93,5 +93,5 @@
           <always_on>true</always_on>
           <pose>0 0 0 0 0 0</pose>
-          <visualize>false</visualize>
+          <visualize>true</visualize>
           <update_rate>${update_rate}</update_rate>
           <ray>
@@ -111,9 +111,8 @@
           </ray>
           <plugin name="gazebo_ros_laser" filename="libgazebo_ros_laser.so">
+            <alwaysOn>true</alwaysOn>
             <topicName>${topic}</topicName>
             <frameName>${frame}</frameName>
-            <robotNamespace>${robot_namespace}</robotNamespace>
             <gaussianNoise>0.005</gaussianNoise>
-            <alwaysOn>true</alwaysOn>
           </plugin>
         </sensor>

File: Task_1/volta_description/urdf/volta.urdf.xacro (robot description, xacro)
@@ -34,6 +34,6 @@
     <xacro:arg name="robot_namespace" default="/" />
     <xacro:arg name="tf_pre"  default= ""/>
-    <xacro:arg name="lidar_enabled" default="false"/>
-    <xacro:arg name="rplidar_a3_enabled" default="false"/>
+    <xacro:arg name="lidar_enabled" default="true"/>
+    <xacro:arg name="rplidar_a3_enabled" default="true"/>
     <xacro:arg name="hokuyo_ust_10lx_enabled" default="false"/>
     <xacro:arg name="imu_enabled" default="true"/>
@@ -102,8 +102,8 @@
         </xacro:if>
         <!-- LIDAR -->
-        <!--xacro:if value="$(arg lidar_enabled)">
+        <xacro:if value="$(arg lidar_enabled)">
             <xacro:include filename="$(find volta_description)/urdf/accessories/lidar_volta.urdf.xacro"/>
-            <xacro:lidar rplidar_a3_enabled="$(arg rplidar_a3_enabled)" hokuyo_ust_10lx_enabled="$(arg hokuyo_ust_10lx_enabled)" robot_namespace="$(arg robot_namespace)">  </xacro:lidar>
-        </xacro:if-->
+            <xacro:lidar rplidar_a3_enabled="$(arg rplidar_a3_enabled)" hokuyo_ust_10lx_enabled="$(arg hokuyo_ust_10lx_enabled)" robot_namespace="$(arg robot_namespace)" ></xacro:lidar>
+        </xacro:if>
         <!--Camera -->
         <!--xacro:if value="$(arg camera_enabled)">
@@ -118,4 +118,24 @@
             </plugin>
         </gazebo>
+        <gazebo>
+         <plugin name="differential_drive_controller" filename="libgazebo_ros_diff_drive.so">
+            <publish_tf>1</publish_tf>
+	    <alwaysOn>true</alwaysOn>
+	    <updateRate>20</updateRate>
+	    <leftJoint>right_wheel_joint</leftJoint>
+    	    <rightJoint>left_wheel_joint</rightJoint>
+	    <wheelSeparation>0.3208</wheelSeparation>
+	    <wheelDiameter>0.085</wheelDiameter>
+	    <commandTopic>cmd_vel</commandTopic>
+	    <odometryTopic>odom</odometryTopic>
+	    <odometryFrame>odom</odometryFrame>
+	    <robotBaseFrame>base_link</robotBaseFrame>
+	    <publish_odom>true</publish_odom>
+            <publish_odom_tf>true</publish_odom_tf>
+            <publish_wheel_tf>true</publish_wheel_tf>
+	    <publishWheelJointState>true</publishWheelJointState>
+	    <legacyMode>true</legacyMode>
+	  </plugin>
+	</gazebo>
     </xacro:macro>
 </robot>

File: Task_1/volta_description/urdf/volta_properties.xacro (robot description, xacro)
@@ -72,6 +72,6 @@
     <xacro:property name="caster_joint_z" value="-0.0008"/>
     <!-- base of lidar mopunt, x position in lidar_volta.urdf.xacro -->
-    <!--xacro:property name="lidar_joint_y" value="0.0"/>
-    <xacro:property name="lidar_joint_z" value="0.1140"/-->
+    <xacro:property name="lidar_joint_y" value="0.0"/>
+    <xacro:property name="lidar_joint_z" value="0.1140"/>
     <!-- base of camera mount -->
     <!--xacro:property name="camera_joint_x" value="0.2285"/>
